File: pcb/board.brd (EAGLE design)
At the start: 102.8 x 96.5 mm, 53 parts, among them X1 PN61729-S

Commit message: Final version of PCB
Parts:
- removed LED_ACTIVE, LED_LCD, LED_ON: (no value), LilyPad-Wearables:LED-1206
- removed R5, R6, R7: 580, rcl:R1206
- added BTN_IN: (no value), con-lstb:MA03-1
- added LED_OUT: (no value), con-lstb:MA04-1
- C14, C15: device resistor:C1206 -> resistor:C025-024X044
- C6: device resistor:C1206 -> resistor:C025-025X050
- LED_RX, LED_TX: device LilyPad-Wearables:LED-1206 -> led:LD260
- moved C6 43.3 mm to (73.7, 35.6), flipped to the top
- moved R3 18.0 mm to (62.2, 9.84)
- moved C8 17.8 mm to (58.7, 74.3), turned to 180 degrees
- moved C5 13.2 mm to (99.1, 14.6)
- moved LED_RX 12.4 mm to (60.6, 14.6), flipped to the top, turned to 270 degrees
- moved C18 9.23 mm to (60.6, 92.4)
- moved LED_TX 5.72 mm to (63.8, 14.6), flipped to the top, turned to 270 degrees
- moved X1 5.08 mm to (92.7, 5.08)
- moved R4 4.58 mm to (67.3, 14.0), turned to 90 degrees
- moved C3 1.91 mm to (80.0, 27.3)
- moved C4 1.91 mm to (80.0, 14.6)
- moved R2 1.91 mm to (76.2, 13.3)
- moved C13 1.90 mm to (21.3, 33.3), turned to 270 degrees
- moved C2 1.90 mm to (76.2, 21.0)
- moved R1 1.90 mm to (76.2, 28.6)
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Connections:
- removed net N$14: LED_LCD.A, R7.2
- removed net N$15: LED_ACTIVE.A, R6.2
- removed net N$16: LED_ON.A, R5.2
- removed net N$18: BTN_DOWN.1, BTN_DOWN.2, R12.2
- removed net N$19: BTN_UP.1, BTN_UP.2, R10.2
- new net DOWN_IN: BTN_DOWN.1, BTN_DOWN.2, BTN_IN.2, R12.2
- new net UP_IN: BTN_IN.1, BTN_UP.1, BTN_UP.2, R10.2
- net ADC_0: now also PGA_0.1; no longer PGA_1.1
- net ADC_1: now also PGA_1.1; no longer PGA_0.1
- net CS_PGA_0: now also MAIN_UC.15; no longer MAIN_UC.12
- net CS_PGA_1: now also MAIN_UC.14; no longer MAIN_UC.13
- net GND: now also BTN_IN.3, LED_OUT.4; no longer LED_ACTIVE.C, LED_LCD.C, LED_ON.C
- net LED_ACTIVE: now also LED_OUT.2, MAIN_UC.13; no longer MAIN_UC.14, R6.1
- net LED_LCD: now also LED_OUT.3, MAIN_UC.12; no longer MAIN_UC.15, R7.1
- net N$1: now also LED_TX.K; no longer LED_TX.C
- net N$3: now also LED_RX.K; no longer LED_RX.C
- net RXD: now also MAIN_UC.3; no longer MAIN_UC.2
- net TXD: now also MAIN_UC.2; no longer MAIN_UC.3
- net VCC: now also LED_OUT.1; no longer R5.1
Routing:
- net LED_LCD: track 74.6 -> 22.8 mm
- net CS_PGA_0: track 87.6 -> 52.1 mm
- net DOWN_IN: track 0.00 -> 31.2 mm
- net VCC: track 609.7 -> 640.5 mm, vias 18 -> 20
- net RX_ON: track 5.37 -> 30.6 mm, vias 0 -> 2
- net GND: track 974.2 -> 996.9 mm, vias 10 -> 14
- net ADC_1: track 57.5 -> 36.4 mm, vias 2 -> 0
- net ADC_0: track 33.4 -> 53.4 mm, vias 0 -> 2
- net UP_IN: track 0.00 -> 18.8 mm
- net VCCIO: track 52.5 -> 64.0 mm
- net N$19: track 10.1 -> 0.00 mm
- net N$18: track 10.1 -> 0.00 mm
- net TX_ON: track 10.2 -> 2.98 mm
- net D-: track 15.9 -> 22.8 mm, vias 0 -> 2
- net CS_PGA_1: track 75.6 -> 70.5 mm
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Other:
- board size 102.8 x 96.5 mm -> 110.5 x 96.5 mm
- board text added: "GND"
- board text added: "MISO"
- board text added: "MOSI"
- board text added: "RESET"
- board text added: "SCK"
- board text added: "VCC"

Commit message: Correct PCB
Parts:
- added C9: 10n, resistor:C1206
Connections:
- new net N$14: C9.1, MAIN_UC.21
- net GND: now also C9.2; no longer MAIN_UC.21
Routing:
- net N$14: track 0.00 -> 4.95 mm
- net GND: track 996.9 -> 995.3 mm
Changed lines of the file:
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@@
 <attribute name="OC_FARNELL" value="unknown" x="6.6675" y="8.255" size="1.778" layer="27" rot="R270" display="off"/>
 </element>
+<element name="C9" library="resistor" package="C1206" value="10n" x="35.56" y="59.69" rot="MR90"/>
 </elements>
 <signals>
@@
 <contactref element="MAIN_UC" pad="8"/>
 <contactref element="MAIN_UC" pad="22"/>
-<contactref element="MAIN_UC" pad="21"/>
 <contactref element="C10" pad="2"/>
 <contactref element="C17" pad="2"/>
@@
 <wire x1="35.69" y1="38.1" x2="35.56" y2="38.1" width="1.016" layer="16"/>
 <wire x1="35.56" y1="38.1" x2="35.56" y2="45.72" width="1.016" layer="16"/>
-<wire x1="35.56" y1="45.72" x2="35.56" y2="49.53" width="1.4224" layer="16"/>
+<wire x1="35.56" y1="45.72" x2="35.56" y2="49.53" width="1.016" layer="16"/>
 <wire x1="7.62" y1="90.17" x2="10.16" y2="90.17" width="1.016" layer="16"/>
 <wire x1="10.16" y1="90.17" x2="12.7" y2="90.17" width="1.016" layer="16"/>
@@
 <wire x1="38.1" y1="94.9325" x2="38.1" y2="95.25" width="1.016" layer="16"/>
 <wire x1="38.1" y1="95.25" x2="46.355" y2="95.25" width="1.016" layer="16"/>
-<wire x1="34.29" y1="68.58" x2="34.29" y2="58.42" width="1.016" layer="16"/>
-<wire x1="34.29" y1="58.42" x2="35.56" y2="56.515" width="1.016" layer="16"/>
-<wire x1="35.56" y1="56.515" x2="35.56" y2="53.34" width="1.016" layer="16"/>
-<wire x1="34.29" y1="68.58" x2="31.75" y2="68.58" width="1.4224" layer="16"/>
+<wire x1="35.56" y1="63.5" x2="31.75" y2="68.58" width="1.4224" layer="16"/>
 <via x="31.75" y="68.58" extent="1-16" drill="0.9" diameter="1.016"/>
 <wire x1="31.75" y1="68.58" x2="31.75" y2="77.47" width="1.016" layer="1"/>
@@
 <via x="15.24" y="49.53" extent="1-16" drill="0.9" diameter="1.016"/>
 <wire x1="15.24" y1="49.53" x2="5.08" y2="49.53" width="1.016" layer="1"/>
-<wire x1="35.56" y1="53.34" x2="35.56" y2="49.53" width="1.4224" layer="16"/>
 <wire x1="35.56" y1="49.53" x2="33.02" y2="49.53" width="1.4224" layer="16"/>
-<wire x1="33.02" y1="49.53" x2="33.02" y2="53.34" width="1.4224" layer="16"/>
+<wire x1="33.02" y1="49.53" x2="33.02" y2="53.34" width="1.016" layer="16"/>
 <via x="5.08" y="49.53" extent="1-16" drill="0.9" diameter="1.016"/>
 <wire x1="96.52" y1="35.8775" x2="96.8375" y2="35.8775" width="1.016" layer="16"/>
@@
 <via x="2.8575" y="14.9225" extent="1-16" drill="0.9"/>
 <wire x1="2.8575" y1="14.9225" x2="-1.27" y2="14.9225" width="1.4224" layer="16"/>
+<contactref element="C9" pad="2"/>
+<wire x1="35.56" y1="63.5" x2="35.56" y2="61.09" width="1.4224" layer="16"/>
+<wire x1="33.02" y1="53.34" x2="33.02" y2="62.23" width="1.016" layer="16"/>
+<wire x1="33.02" y1="62.23" x2="34.925" y2="64.135" width="1.016" layer="16"/>
 </signal>
 <signal name="N$2">
@@
 <wire x1="60.808" y1="9.525" x2="60.808" y2="9.8425" width="1.016" layer="16"/>
 </signal>
+<signal name="N$14">
+<contactref element="MAIN_UC" pad="21"/>
+<contactref element="C9" pad="1"/>
+<wire x1="35.56" y1="58.29" x2="35.56" y2="53.34" width="1.016" layer="16"/>
+</signal>
 </signals>
