File: pcb/board.sch (EAGLE design)
At the start: 15 parts

Commit message: Upgrade board
Parts:
- added AIN, GND, VCC: (no value), con-lstb:MA06-1
- added C10, C11, C7, C8, C9: 100n, resistor:C-EUC1206
- added DOUT: (no value), con-lstb:MA08-2
- added LCD_0: LPH-7366, lph-7366:LPH-7366
- added PGA_0, PGA_1: MCP6S21I/SN, MPC6S21:MCP6S21I/SN
- added SHR_0: 74HC595D, 74xx-eu:74HC595D
- added U$1: AVR_SPI_PRG_6PTH, SparkFun:AVR_SPI_PRG_6PTH
Connections:
- new net ADC_0: MAIN_UC.PC0(ADC0), PGA_0.VOUT
- new net ADC_1: MAIN_UC.PC1(ADC1), PGA_1.VOUT
- new net ADC_2: AIN.3, MAIN_UC.PC2(ADC2)
- new net ADC_3: AIN.4, MAIN_UC.PC3(ADC3)
- new net ADC_4: AIN.5, MAIN_UC.PC4(ADC4/SDA)
- new net ADC_5: AIN.6, MAIN_UC.PC5(ADC5/SCL)
- new net AIN_0: AIN.1, PGA_0.CH0
- new net AIN_1: AIN.2, PGA_1.CH0
- new net CS_LCD_0: LCD_0./SCE, MAIN_UC.PD4(XCK/T0)
- new net CS_PGA_0: MAIN_UC.PD6(AIN0), PGA_0./CS
- new net CS_PGA_1: MAIN_UC.PD7(AIN1), PGA_1./CS
- new net CS_SHR_0: MAIN_UC.PD5(T1)
- new net INT_0: MAIN_UC.PD2(INT0)
- new net INT_1: MAIN_UC.PD3(INT1)
- new net LED_ACTIVE: MAIN_UC.PB0(ICP)
- new net LED_LCD: MAIN_UC.PB1(OC1A)
- new net MISO: MAIN_UC.PB4(MISO)
- new net MOSI: LCD_0.SDIN, MAIN_UC.PB3(MOSI/OC2), PGA_0.SI, PGA_1.SI, SHR_0A.SER
- new net N$10: DOUT.8, SHR_0A.QE
- new net N$11: DOUT.6, SHR_0A.QF
- new net N$12: DOUT.4, SHR_0A.QG
- new net N$13: DOUT.2, SHR_0A.QH
- new net N$4: DOUT.16, SHR_0A.QA
- new net N$7: DOUT.14, SHR_0A.QB
- new net N$8: DOUT.12, SHR_0A.QC
- new net N$9: DOUT.10, SHR_0A.QD
- new net RESET: MAIN_UC.PC6(/RESET)
- new net SCK: LCD_0.SCLK, MAIN_UC.PB5(SCK), PGA_0.SCK, PGA_1.SCK, SHR_0A.SCK
- new net SHR_CK: MAIN_UC.PB2(SS/OC1B), SHR_0A.G, SHR_0A.RCK
- new net XTAL1: MAIN_UC.PB6(XTAL1/TOSC1)
- new net XTAL2: MAIN_UC.PB7(XTAL2/TOSC2)
- net GND: now also C10.2, C11.2, C7.2, C8.2, C9.2, DOUT.1, DOUT.11, DOUT.13, DOUT.15, DOUT.3, DOUT.5, DOUT.7, DOUT.9, GND.1, GND.2, GND.3, GND.4, GND.5, GND.6, LCD_0.GND, MAIN_UC.AREF, MAIN_UC.GND@1, MAIN_UC.GND@2, PGA_0.VREF, PGA_0.VSS, PGA_1.VREF, PGA_1.VSS, SHR_0P.GND
- net VCC: now also C10.1, C11.1, C7.1, C8.1, C9.1, LCD_0./RES, LCD_0.D/C, LCD_0.OSC, LCD_0.VDD, MAIN_UC.AVCC, MAIN_UC.VCC, PGA_0.VDD, PGA_1.VDD, SHR_0A.SCL, SHR_0P.VCC, VCC.1, VCC.2, VCC.3, VCC.4, VCC.5, VCC.6

Commit message: Add complete PCB
Parts:
- removed C9: 100n, resistor:C-EUC1206
- removed LCD_0: LPH-7366, lph-7366:LPH-7366
- removed RX_LED, TX_LED: (no value), LilyPad-Wearables:LED1206
- removed U$1: AVR_SPI_PRG_6PTH, SparkFun:AVR_SPI_PRG_6PTH
- removed USB: USB_B_SCHIELDED, con-cypressindustries:MINI-USB_SHIELD4P-85-32004-30X-1
- added 20MHZ: (no value), crystal:CRYSTALHC49S
- added BTN_DOWN, BTN_UP, RESET_SW: (no value), switch-omron:10-XX
- added C12, C13, C18: 100n, resistor:C-EUC1206
- added C14, C15: 1u, resistor:C-EUC1206
- added C16, C17: 12p, resistor:C-EUC1206
- added LCD_OUT: (no value), con-lstb:MA05-1
- added LED_ACTIVE, LED_LCD, LED_ON, LED_RX, LED_TX: (no value), LilyPad-Wearables:LED1206
- added NOT_0, NOT_1: 74LVC1G14DCK, 74xx-little-us:74LVC1G14DCK
- added PROG: AVR_SPI_PRG, SparkFun:AVR_SPI_PRG_6PTH
- added R10, R12: 100, rcl:R-EU_R1206
- added R11, R9: 10k, rcl:R-EU_R1206
- added R5, R6, R7: 580, rcl:R-EU_R1206
- added R8: 5k, rcl:R-EU_R1206
- added RESET_GEN: DS1813-SMD, ds1813_revised:DS1813-SMD
- added X1: PN61729-S, con-berg:PN61729-S
Connections:
- removed net SHR_CK: MAIN_UC.PB2(SS/OC1B), SHR_0A.G, SHR_0A.RCK
- new net N$14: LED_LCD.A, R7.2
- new net N$15: LED_ACTIVE.A, R6.2
- new net N$16: LED_ON.A, R5.2
- new net N$17: R8.1, RESET_GEN./RST, RESET_SW.P, RESET_SW.P1
- new net N$18: BTN_DOWN.S, BTN_DOWN.S1, R12.2
- new net N$19: BTN_UP.S, BTN_UP.S1, R10.2
- new net N$20: C14.1, NOT_0A.I, R10.1, R9.1
- new net N$21: C15.1, NOT_1A.I, R11.1, R12.1
- new net SS: MAIN_UC.PB2(SS/OC1B)
- net ADC_0: now also PGA_1.VOUT; no longer PGA_0.VOUT
- net ADC_1: now also PGA_0.VOUT; no longer PGA_1.VOUT
- net CS_LCD_0: now also LCD_OUT.2; no longer LCD_0./SCE
- net CS_SHR_0: now also SHR_0A.G, SHR_0A.RCK
- net D+: now also X1.3
- net D-: now also X1.2
- net GND: now also BTN_DOWN.P, BTN_DOWN.P1, BTN_UP.P, BTN_UP.P1, C12.2, C13.2, C14.2, C15.2, C16.2, C17.2, C18.2, LCD_OUT.1, LED_ACTIVE.C, LED_LCD.C, LED_ON.C, NOT_0P.GND, NOT_1P.GND, PROG.6, RESET_GEN.GND, RESET_SW.S, RESET_SW.S1, X1.4, X1.S1, X1.S2; no longer C9.2, LCD_0.GND, USBS.S1, USBS.S2
- net INT_0: now also NOT_0A.O
- net INT_1: now also NOT_1A.O
- net LED_ACTIVE: now also R6.1
- net LED_LCD: now also R7.1
- net MISO: now also PROG.1
- net MOSI: now also LCD_OUT.4, PROG.4; no longer LCD_0.SDIN
- net N$1: now also LED_TX.C; no longer TX_LED.C
- net N$3: now also LED_RX.C; no longer RX_LED.C
- net RESET: now also PROG.5, R8.2
- net SCK: now also LCD_OUT.3, PROG.3; no longer LCD_0.SCLK
- net VCC: now also C12.1, C13.1, C18.1, LCD_OUT.5, NOT_0P.VCC, NOT_1P.VCC, PROG.2, R11.2, R5.1, R9.2, RESET_GEN.+5V, X1.1; no longer C9.1, LCD_0./RES, LCD_0.D/C, LCD_0.OSC, LCD_0.VDD
- net VCCIO: now also LED_RX.A, LED_TX.A; no longer RX_LED.A, TX_LED.A
- net XTAL1: now also 20MHZ.2, C17.1
- net XTAL2: now also 20MHZ.1, C16.1
Other:
- moved on the sheet: AIN, C1, C10, C11, C2, C3, C4, C5, C6, C7, C8, DOUT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

Commit message: Final version of PCB
Parts:
- removed LED_ACTIVE, LED_LCD, LED_ON: (no value), LilyPad-Wearables:LED1206
- removed R5, R6, R7: 580, rcl:R-EU_R1206
- added BTN_IN: (no value), con-lstb:MA03-1
- added LED_OUT: (no value), con-lstb:MA04-1
- C14, C15: device resistor:C-EUC1206 -> resistor:C-EU025-024X044
- C6: device resistor:C-EUC1206 -> resistor:C-EU025-025X050
- LED_RX, LED_TX: device LilyPad-Wearables:LED1206 -> led:LEDLD260
Connections:
- removed net N$14: LED_LCD.A, R7.2
- removed net N$15: LED_ACTIVE.A, R6.2
- removed net N$16: LED_ON.A, R5.2
- removed net N$18: BTN_DOWN.S, BTN_DOWN.S1, R12.2
- removed net N$19: BTN_UP.S, BTN_UP.S1, R10.2
- new net DOWN_IN: BTN_DOWN.S, BTN_DOWN.S1, BTN_IN.2, R12.2
- new net UP_IN: BTN_IN.1, BTN_UP.S, BTN_UP.S1, R10.2
- net ADC_0: now also PGA_0.VOUT; no longer PGA_1.VOUT
- net ADC_1: now also PGA_1.VOUT; no longer PGA_0.VOUT
- net CS_PGA_0: now also MAIN_UC.PB1(OC1A); no longer MAIN_UC.PD6(AIN0)
- net CS_PGA_1: now also MAIN_UC.PB0(ICP); no longer MAIN_UC.PD7(AIN1)
- net GND: now also BTN_IN.3, LED_OUT.4; no longer LED_ACTIVE.C, LED_LCD.C, LED_ON.C
- net LED_ACTIVE: now also LED_OUT.2, MAIN_UC.PD7(AIN1); no longer MAIN_UC.PB0(ICP), R6.1
- net LED_LCD: now also LED_OUT.3, MAIN_UC.PD6(AIN0); no longer MAIN_UC.PB1(OC1A), R7.1
- net RXD: now also MAIN_UC.PD1(TXD); no longer MAIN_UC.PD0(RXD)
- net TXD: now also MAIN_UC.PD0(RXD); no longer MAIN_UC.PD1(TXD)
- net VCC: now also LED_OUT.1; no longer R5.1
Other:
- moved on the sheet: BTN_DOWN, BTN_UP, C14, C15, LED_TX, NOT_0, NOT_1, R10, R11, R12, R4, R9

Commit message: Correct PCB
Parts:
- added C9: 10n, resistor:C-EUC1206
Connections:
- new net N$14: C9.1, MAIN_UC.AREF
- net GND: now also C9.2; no longer MAIN_UC.AREF
Changed lines of the file:
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@@
 <part name="BTN_IN" library="con-lstb" deviceset="MA03-1" device=""/>
 <part name="GND4" library="supply1" deviceset="GND" device=""/>
+<part name="C9" library="resistor" deviceset="C-EU" device="C1206" value="10n"/>
 </parts>
 <sheets>
@@
 <instance part="BTN_IN" gate="G$1" x="30.48" y="-157.48" rot="R180"/>
 <instance part="GND4" gate="1" x="7.62" y="-165.1"/>
+<instance part="C9" gate="G$1" x="73.66" y="-22.86" rot="R270"/>
 </instances>
 <busses>
@@
 <wire x1="78.74" y1="-63.5" x2="63.5" y2="-63.5" width="0.1524" layer="91"/>
 <junction x="63.5" y="-63.5"/>
-<pinref part="MAIN_UC" gate="G$1" pin="AREF"/>
-<wire x1="78.74" y1="-22.86" x2="63.5" y2="-22.86" width="0.1524" layer="91"/>
 <wire x1="63.5" y1="-22.86" x2="63.5" y2="-45.72" width="0.1524" layer="91"/>
 <junction x="63.5" y="-60.96"/>
 <pinref part="C10" gate="G$1" pin="2"/>
-<junction x="63.5" y="-22.86"/>
 <pinref part="C17" gate="G$1" pin="2"/>
 <wire x1="63.5" y1="-45.72" x2="63.5" y2="-60.96" width="0.1524" layer="91"/>
@@
 <junction x="22.86" y="-45.72"/>
 <junction x="63.5" y="-45.72"/>
+<pinref part="C9" gate="G$1" pin="2"/>
+<wire x1="68.58" y1="-22.86" x2="63.5" y2="-22.86" width="0.1524" layer="91"/>
+<junction x="63.5" y="-22.86"/>
 </segment>
 <segment>
@@
 </segment>
 </net>
+<net name="N$14" class="0">
+<segment>
+<pinref part="MAIN_UC" gate="G$1" pin="AREF"/>
+<pinref part="C9" gate="G$1" pin="1"/>
+<wire x1="78.74" y1="-22.86" x2="76.2" y2="-22.86" width="0.1524" layer="91"/>
+</segment>
+</net>
